Commit message: to work with ign gazebo

File: interbotix_ros_xslocobots/interbotix_xslocobot_descriptions/urdf/arms/arm_control.urdf.xacro (robot description, xacro)
@@ -18,4 +18,7 @@
       <xacro:if value="${hardware_type == 'gz_classic'}">
         <plugin>gazebo_ros2_control/GazeboSystem</plugin>
+      </xacro:if>
+      <xacro:if value="${hardware_type == 'gz_ignition'}">
+        <plugin>gz_ros2_control/GazeboSimSystem</plugin>
       </xacro:if>
     </hardware>
@@ -88,5 +91,5 @@
           <param name="initial_position">0.0195</param>
         </joint>
-        <xacro:if value="${hardware_type == 'gz_classic'}">
+        <xacro:if value="${hardware_type in ('gz_classic', 'gz_ignition')}">
           <joint name="right_finger">
             <!-- <param name="mimic">left_finger</param>

File: interbotix_ros_xslocobots/interbotix_xslocobot_descriptions/urdf/create3_version/locobot_create3.urdf.xacro (robot description, xacro)
@@ -1,15 +1,4 @@
 <?xml version="1.0" ?>
 <robot xmlns:xacro="http://ros.org/wiki/xacro">
-    <!-- Much of the following iRobot Create3 description is taken from https://github.com/iRobotEducation/create3_sim/tree/6b8a4a6ce0d0902a7de117c29cbe55bfc52a4e54/irobot_create_common/irobot_create_description/urdf -->
-    <!-- The original 3-Clause BSD License is retained below -->
-    <!--
-      Copyright 2021 iRobot Corporation.
-      Redistribution and use in source and binary forms, with or without modification, are permitted provided that the following conditions are met:
-      1. Redistributions of source code must retain the above copyright notice, this list of conditions and the following disclaimer.
-      2. Redistributions in binary form must reproduce the above copyright notice, this list of conditions and the following disclaimer in the documentation and/or other materials provided with the distribution.
-      3. Neither the name of the copyright holder nor the names of its contributors may be used to endorse or promote products derived from this software without specific prior written permission.
-      THIS SOFTWARE IS PROVIDED BY THE COPYRIGHT HOLDERS AND CONTRIBUTORS "AS IS" AND ANY EXPRESS OR IMPLIED WARRANTIES, INCLUDING, BUT NOT LIMITED TO, THE IMPLIED WARRANTIES OF MERCHANTABILITY AND FITNESS FOR A PARTICULAR PURPOSE ARE DISCLAIMED.
-      IN NO EVENT SHALL THE COPYRIGHT HOLDER OR CONTRIBUTORS BE LIABLE FOR ANY DIRECT, INDIRECT, INCIDENTAL, SPECIAL, EXEMPLARY, OR CONSEQUENTIAL DAMAGES (INCLUDING, BUT NOT LIMITED TO, PROCUREMENT OF SUBSTITUTE GOODS OR SERVICES; LOSS OF USE, DATA, OR PROFITS; OR BUSINESS INTERRUPTION) HOWEVER CAUSED AND ON ANY THEORY OF LIABILITY, WHETHER IN CONTRACT, STRICT LIABILITY, OR TORT (INCLUDING NEGLIGENCE OR OTHERWISE) ARISING IN ANY WAY OUT OF THE USE OF THIS SOFTWARE, EVEN IF ADVISED OF THE POSSIBILITY OF SUCH DAMAGE.
-    -->
     <xacro:include filename="$(find interbotix_xslocobot_descriptions)/urdf/create3_version/bumper.urdf.xacro" />
     <xacro:include filename="$(find interbotix_xslocobot_descriptions)/urdf/create3_version/bump_caster.urdf.xacro" />
@@ -50,5 +39,5 @@
       <xacro:property name="caster_position_z"       value="${-5.2*cm2m}" />
     </xacro:if>
-    <xacro:property name="wheel_drop_offset_z"     value="${3.5*mm2m}"/>
+    <xacro:property name="wheel_drop_offset_z"     value="${0.5*mm2m}"/>
     <xacro:property name="wheel_drop_z"            value="${wheel_height + wheel_drop_offset_z}"/>
     <xacro:property name="base_link_z_offset"     value="${6.42*cm2m}"/>

File: interbotix_ros_xslocobots/interbotix_xslocobot_descriptions/urdf/create3_version/wheel.urdf.xacro (robot description, xacro)
@@ -53,5 +53,5 @@
     <ros2_control name="${robot_name}/${wheel_link_name}_controller" type="system">
       <hardware>
-        <plugin>ign_ros2_control/IgnitionSystem</plugin>
+        <plugin>gz_ros2_control/GazeboSimSystem</plugin>
       </hardware>
       <joint name="${wheel_joint_name}">
